File: arduino_duo_shield/Spindle_Power_Control.sch (KiCad schematic (older format))
At the start: 11 parts, among them J1 Spindle_Power, K1 G5Q-1, Q2 IRFZ44N, U3 PC817, U5 PC817

Commit message: Power block to PCB
Parts:
- C1: footprint Capacitor_THT:C_Disc_D5.0mm_W2.5mm_P2.50mm -> Capacitor_THT:CP_Radial_D5.0mm_P2.50mm; symbol Device:C_Small -> Device:CP1
- J1: footprint Connector_PinHeader_2.54mm:PinHeader_1x02_P2.54mm_Vertical -> TerminalBlock_RND:TerminalBlock_RND_205-00276_1x02_P5.00mm_Vertical
- R1, R16, R17, R2: footprint Resistor_THT:R_Axial_DIN0204_L3.6mm_D1.6mm_P2.54mm_Vertical -> Resistor_THT:R_Axial_DIN0204_L3.6mm_D1.6mm_P5.08mm_Horizontal
Connections:
- net +24V: no longer U3.4
- net at C1.1, D1.2 (A), K1.2: now also J1.2 (Pin_2), U3.4; no longer J1.1 (Pin_1)
- net at C1.2, D1.1 (K), Q2.2 (D): now also J1.1 (Pin_1); no longer J1.2 (Pin_2)
Changed lines of the file:
@@
 $Descr A4 11693 8268
 encoding utf-8
-Sheet 2 3
+Sheet 3 3
 Title ""
 Date ""
@@
 $EndComp
 $Comp
-L Device:C_Small C1
+L Device:CP1 C1
 U 1 1 5D7E3901
 P 5600 5300
 F 0 "C1" H 5692 5346 50  0000 L CNN
 F 1 "100u" H 5692 5255 50  0000 L CNN
-F 2 "Capacitor_THT:C_Disc_D5.0mm_W2.5mm_P2.50mm" H 5600 5300 50  0001 C CNN
+F 2 "Capacitor_THT:CP_Radial_D5.0mm_P2.50mm" H 5600 5300 50  0001 C CNN
 F 3 "~" H 5600 5300 50  0001 C CNN
 	1    5600 5300
@@
 $EndComp
 Wire Wire Line
-	5600 5200 5600 5000
+	5600 5150 5600 5000
 $Comp
 L Transistor_FET:IRLZ44N Q?
@@
 F 0 "R1" H 3220 6296 50  0000 L CNN
 F 1 "220" H 3220 6205 50  0000 L CNN
-F 2 "Resistor_THT:R_Axial_DIN0204_L3.6mm_D1.6mm_P2.54mm_Vertical" V 3080 6250 50  0001 C CNN
+F 2 "Resistor_THT:R_Axial_DIN0204_L3.6mm_D1.6mm_P5.08mm_Horizontal" V 3080 6250 50  0001 C CNN
 F 3 "~" H 3150 6250 50  0001 C CNN
 	1    3150 6250
@@
 F 0 "R2" H 4770 6746 50  0000 L CNN
 F 1 "1.5K" H 4770 6655 50  0000 L CNN
-F 2 "Resistor_THT:R_Axial_DIN0204_L3.6mm_D1.6mm_P2.54mm_Vertical" V 4630 6700 50  0001 C CNN
+F 2 "Resistor_THT:R_Axial_DIN0204_L3.6mm_D1.6mm_P5.08mm_Horizontal" V 4630 6700 50  0001 C CNN
 F 3 "~" H 4700 6700 50  0001 C CNN
 	1    4700 6700
@@
 Wire Wire Line
 	3300 6250 3350 6250
-$Comp
-L Connector:Conn_01x02_Male J1
-U 1 1 5D7E3942
-P 6200 5250
-F 0 "J1" H 6172 5224 50  0000 R CNN
-F 1 "Spindle_Power" H 6172 5133 50  0000 R CNN
-F 2 "Connector_PinHeader_2.54mm:PinHeader_1x02_P2.54mm_Vertical" H 6200 5250 50  0001 C CNN
-F 3 "~" H 6200 5250 50  0001 C CNN
-	1    6200 5250
-	-1   0    0    -1
-$EndComp
 Wire Wire Line
 	5100 5600 5600 5600
@@
 	5100 5500 5100 5600
 Wire Wire Line
-	5600 5400 5600 5600
+	5600 5450 5600 5600
 Connection ~ 5600 5600
 Wire Wire Line
@@
 	3300 3950 3300 4050
 Wire Wire Line
-	5100 5000 3400 5000
+	5100 5000 4200 5000
 Wire Wire Line
 	3400 5000 3400 4650
@@
 F 0 "R16" H 4770 7246 50  0000 L CNN
 F 1 "1K" H 4770 7155 50  0000 L CNN
-F 2 "Resistor_THT:R_Axial_DIN0204_L3.6mm_D1.6mm_P2.54mm_Vertical" V 4630 7200 50  0001 C CNN
+F 2 "Resistor_THT:R_Axial_DIN0204_L3.6mm_D1.6mm_P5.08mm_Horizontal" V 4630 7200 50  0001 C CNN
 F 3 "~" H 4700 7200 50  0001 C CNN
 	1    4700 7200
@@
 Wire Wire Line
 	3950 6250 4200 6250
-Wire Wire Line
-	4200 6250 4200 3950
-Connection ~ 4200 3950
 Wire Wire Line
 	2400 5200 2400 7500
@@
 F 0 "R17" H 2270 5046 50  0000 L CNN
 F 1 "220" H 2270 4955 50  0000 L CNN
-F 2 "Resistor_THT:R_Axial_DIN0204_L3.6mm_D1.6mm_P2.54mm_Vertical" V 2130 5000 50  0001 C CNN
+F 2 "Resistor_THT:R_Axial_DIN0204_L3.6mm_D1.6mm_P5.08mm_Horizontal" V 2130 5000 50  0001 C CNN
 F 3 "~" H 2200 5000 50  0001 C CNN
 	1    2200 5000
@@
 Wire Wire Line
 	3000 5200 3000 7500
+Wire Wire Line
+	4200 6250 4200 5000
+Connection ~ 4200 5000
+Wire Wire Line
+	4200 5000 3400 5000
+$Comp
+L Connector:Conn_01x02_Male J1
+U 1 1 5D7E3942
+P 6200 5350
+F 0 "J1" H 6172 5324 50  0000 R CNN
+F 1 "Spindle_Power" H 6172 5233 50  0000 R CNN
+F 2 "TerminalBlock_RND:TerminalBlock_RND_205-00276_1x02_P5.00mm_Vertical" H 6200 5350 50  0001 C CNN
+F 3 "~" H 6200 5350 50  0001 C CNN
+	1    6200 5350
+	-1   0    0    1
+$EndComp
 $EndSCHEMATC

Commit message: Add PCB front/back for spindle controls
Parts:
- added D2: 1N4007, Diode_THT:D_A-405_P7.62mm_Horizontal, symbol pspice:DIODE
- added J7: Power_In, TerminalBlock:TerminalBlock_bornier-2_P5.08mm, symbol Connector:Conn_01x02_Male
- added P14, P15, P16, P17: CONN_01X01, Socket_Arduino_Mega:Arduino_1pin, symbol Connector_Generic:Conn_01x01
- D1: value DIODE -> 1N4007
- J1: footprint TerminalBlock_RND:TerminalBlock_RND_205-00276_1x02_P5.00mm_Vertical -> TerminalBlock:TerminalBlock_bornier-2_P5.08mm
- K1: value G5Q-1 -> JQC-3F; footprint Relay_THT:Relay_SPDT_Omron-G5Q-1 -> Relay_THT:Relay_SPDT_SANYOU_SRD_Series_Form_C; symbol Relay:G5Q-1 -> Relay:G5LE-1
- R17: value 220 -> 100
- R2: value 1.5K -> 1.3K
Connections:
- net ext_sppwm is gone; now on net ext_gnd: R1.2
- net ext_gnd: no longer Q2.3 (S), R16.2
- net ext_vcc: now also D2.2 (A)
- net at K1.1: now also C1.1, D1.2 (A), J1.2 (Pin_2), U3.4; no longer U5.4
- net MOTOR_POW_24V: now reaches K1.3
- net MOTOR_POW_24V: now also J7.2 (Pin_2)
- net +24V: no longer names the net of K1.4
- net ext_spena renamed ext_spenab
- new net: D2.1 (K), K1.2, U5.4
- new net MOTOR_GND: J7.1 (Pin_1), Q2.3 (S), R16.2
- no-connect marks 1 -> 5
Other:
- note added: "Holes"
- moved on the sheet: C1, D1, J1, K1, Q2, R1, R16, R17, R2, U3, U5

Commit message: Complete wiring
Parts:
- added Q1: 2N7000, Package_TO_SOT_THT:TO-92_Inline, symbol Transistor_FET:2N7000
- added R18: 10K, Resistor_THT:R_Axial_DIN0204_L3.6mm_D1.6mm_P5.08mm_Horizontal, symbol Device:R
Connections:
- net ext_gnd: now also Q1.1 (S), R18.1; no longer R1.2, U5.3
- net ext_vcc: now also U5.4
- net at D2.1 (K), K1.2: now also Q1.3 (D); no longer U5.4
- new net: Q1.2 (G), R18.2, U5.3
- new net ext_sppwm: R1.2
Other:
- moved on the sheet: R1
Changed lines of the file:
@@
 $Descr A4 11693 8268
 encoding utf-8
-Sheet 3 3
+Sheet 3 4
 Title ""
 Date ""
@@
 	1    0    0    -1
 $EndComp
-Wire Wire Line
-	5050 6050 5050 5000
 $Comp
 L Device:R R1
 U 1 1 5D7E3933
-P 4850 4800
-F 0 "R1" H 4920 4846 50  0000 L CNN
-F 1 "220" H 4920 4755 50  0000 L CNN
-F 2 "Resistor_THT:R_Axial_DIN0204_L3.6mm_D1.6mm_P5.08mm_Horizontal" V 4780 4800 50  0001 C CNN
-F 3 "~" H 4850 4800 50  0001 C CNN
-	1    4850 4800
-	0    1    1    0
-$EndComp
-Wire Wire Line
-	4700 4800 3550 4800
+P 3900 4800
+F 0 "R1" H 3970 4846 50  0000 L CNN
+F 1 "220" H 3970 4755 50  0000 L CNN
+F 2 "Resistor_THT:R_Axial_DIN0204_L3.6mm_D1.6mm_P5.08mm_Horizontal" V 3830 4800 50  0001 C CNN
+F 3 "~" H 3900 4800 50  0001 C CNN
+	1    3900 4800
+	0    1    -1   0
+$EndComp
 $Comp
 L Device:R R2
@@
 $EndComp
 Wire Wire Line
-	5000 4800 5050 4800
-Wire Wire Line
 	6300 4150 6650 4150
 Wire Wire Line
@@
 Wire Wire Line
 	5500 2500 5500 2700
-Text HLabel 3550 6050 0    50   Input ~ 0
+Text HLabel 3550 5000 0    50   Input ~ 0
 ext_gnd
 Text HLabel 3550 4800 0    50   Input ~ 0
 ext_sppwm
 Wire Wire Line
-	3550 6050 4100 6050
+	3550 5000 4100 5000
 Text HLabel 3550 3550 0    50   Input ~ 0
 ext_spenab
@@
 	1    0    0    -1
 $EndComp
-Connection ~ 4700 6050
 Wire Wire Line
 	6300 5700 6300 6050
 Wire Wire Line
 	5900 5000 5900 5100
-Wire Wire Line
-	4700 6050 5050 6050
 $Comp
 L Device:R R16
@@
 	5650 4800 5900 4800
 Wire Wire Line
-	4100 3750 4100 6050
-Connection ~ 4100 6050
-Wire Wire Line
-	4100 6050 4700 6050
+	4100 3750 4100 5000
+Connection ~ 4100 5000
 $Comp
 L Device:R R17
@@
 	5650 5000 5900 5000
 Wire Wire Line
-	4700 3750 4700 4800
-Wire Wire Line
 	5900 4800 5900 3550
 Connection ~ 5900 3550
@@
 	-1   0    0    1
 $EndComp
-Wire Wire Line
-	4700 3550 5050 3550
 $Comp
 L pspice:DIODE D2
@@
 	5900 3550 6300 3550
 Wire Wire Line
-	3550 2500 5050 2500
+	3550 2500 4700 2500
 Connection ~ 5050 3550
 Wire Wire Line
@@
 Text Label 6900 2600 0    50   ~ 0
 MOTOR_GND
-Connection ~ 4700 4800
-Wire Wire Line
-	4700 4800 4700 6050
+$Comp
+L Transistor_FET:2N7000 Q1
+U 1 1 5D7E4BFC
+P 4950 3750
+F 0 "Q1" H 5156 3796 50  0000 L CNN
+F 1 "2N7000" H 5156 3705 50  0000 L CNN
+F 2 "Package_TO_SOT_THT:TO-92_Inline" H 5150 3675 50  0001 L CIN
+F 3 "https://www.fairchildsemi.com/datasheets/2N/2N7000.pdf" H 4950 3750 50  0001 L CNN
+	1    4950 3750
+	1    0    0    -1
+$EndComp
+Wire Wire Line
+	4700 3750 4750 3750
+$Comp
+L Device:R R18
+U 1 1 5D7E83DD
+P 4700 4150
+F 0 "R18" H 4770 4196 50  0000 L CNN
+F 1 "10K" H 4770 4105 50  0000 L CNN
+F 2 "Resistor_THT:R_Axial_DIN0204_L3.6mm_D1.6mm_P5.08mm_Horizontal" V 4630 4150 50  0001 C CNN
+F 3 "~" H 4700 4150 50  0001 C CNN
+	1    4700 4150
+	-1   0    0    1
+$EndComp
+Wire Wire Line
+	4100 5000 4700 5000
+Wire Wire Line
+	4700 3750 4700 4000
+Connection ~ 4700 3750
+Connection ~ 4700 5000
+Wire Wire Line
+	4700 5000 5050 5000
+Wire Wire Line
+	4700 4300 4700 4550
+Wire Wire Line
+	3550 4800 3750 4800
+Wire Wire Line
+	4050 4800 5050 4800
+Wire Wire Line
+	5050 3950 5050 4550
+Wire Wire Line
+	5050 4550 4700 4550
+Connection ~ 4700 4550
+Wire Wire Line
+	4700 4550 4700 5000
+Wire Wire Line
+	4700 2500 4700 3550
+Connection ~ 4700 2500
+Wire Wire Line
+	4700 2500 5050 2500
 $EndSCHEMATC

Commit message: Fix diode symbol in schematic
Parts:
- D1, D2: symbol pspice:DIODE -> Device:D_ALT
Connections:
- net ext_vcc: now also D2.1 (K); no longer D2.2 (A)
- net at C1.1, J1.2 (Pin_2), K1.1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: now also D1.1 (K); no longer D1.2 (A)
- net at K1.2, Q1.3 (D): now also D2.2 (A); no longer D2.1 (K)
- net at C1.2, J1.1 (Pin_1), Q2.2 (D): now also D1.2 (A); no longer D1.1 (K)
- no-connect marks 5 -> 6
Changed lines of the file:
@@
 NoConn ~ 5800 2700
 Wire Wire Line
-	6300 3650 6300 3550
+	6300 3700 6300 3550
 Wire Wire Line
 	4050 3550 4100 3550
 $Comp
-L pspice:DIODE D1
+L Device:D_ALT D1
 U 1 1 5D7E38FB
 P 6300 3850
@@
 F 3 "~" H 6300 3850 50  0001 C CNN
 	1    6300 3850
-	0    -1   -1   0
+	0    -1   1    0
 $EndComp
 $Comp
@@
 	7050 3900 7050 4150
 Wire Wire Line
-	6300 4050 6300 4150
+	6300 4000 6300 4150
 Wire Wire Line
 	6650 4000 6650 4150
@@
 $EndComp
 $Comp
-L pspice:DIODE D2
+L Device:D_ALT D2
 U 1 1 5D88A789
 P 5050 3000
@@
 F 3 "~" H 5050 3000 50  0001 C CNN
 	1    5050 3000
-	0    -1   -1   0
-$EndComp
-Wire Wire Line
-	5050 2500 5050 2800
-Wire Wire Line
-	5050 3200 5050 3550
+	0    -1   1    0
+$EndComp
+Wire Wire Line
+	5050 2500 5050 2850
+Wire Wire Line
+	5050 3150 5050 3550
 $Comp
 L Connector:Conn_01x02_Male J7
@@
 Wire Wire Line
 	4700 2500 5050 2500
+NoConn ~ 7350 1500
 $EndSCHEMATC
